File: usb-audio.brd (EAGLE design)
At the start: 100 x 80 mm, 12 parts

Commit message: .
Parts:
- removed C1, C2, C3: (no value), rcl:A/3216-18R
- added C6: 10mF, rcl:CT3216
- added C7: 100mF, rcl:CT3216
- added IC1: LM1117MPX-3.3, lm1117:SOT223
- added U$3: MICRO-USB, microusb:MICRO-USB
- moved Q1 85.9 mm to (61.8, 18.9)
- moved C4 85.0 mm to (60.5, 11.9)
- moved C5 85.0 mm to (60.5, 5.52)
- moved R2 31.6 mm to (13.0, 13.1)
- moved R1 29.3 mm to (13.0, 16.1)
- moved R4 19.1 mm to (34.3, 28.9)
- moved R3 17.7 mm to (28.5, 28.9)
- moved U$1 15.0 mm to (39.5, 7.05)
- moved U$2 8.06 mm to (26.1, 15.1), turned to 270 degrees
Connections:
- removed net SVSS: U$1.12
- removed net VDD: U$1.2
- new net +3V3: C7.+, IC1.2, IC1.TAB
- new net AGND: U$1.10, U$1.4, U$2.12, U$2.17
- new net GND: C4.2, C5.2, C6.-, C7.-, IC1.1, U$3.5, U$3.GND1, U$3.GND2
- new net N$10: U$1.5
- new net N$11: U$1.9, U$2.14
- new net N$12: U$1.11, U$2.15
- new net N$13: U$1.12, U$1.7
- new net N$5: R1.1, U$3.2
- new net N$6: R2.1, U$3.3
- new net N$7: C5.1, Q1.1, U$2.28
- new net N$8: C4.1, Q1.3, U$2.1
- new net N$9: U$1.3
- new net VCC: C6.+, IC1.3, U$1.2, U$1.8, U$3.1
Other:
- board size 100 x 80 mm -> 54 x 32 mm

Commit message: rev 1
Parts:
- added C1: 100n, rcl:C0805
- added C10, C11, C2, C3, C8: 22, rcl:C0805
- added C12, C13: 220uF, rcl:E2-5
- added C14, C15: 1uf, rcl:C0805
- added C9: 10mF, rcl:CT3216
- added J1: PJ-324MH, audio:PJ-324MH
- added LED1: TLLR4400, led:LED3MM
- added R10, R9: 10k, rcl:R0805
- added R11, R12: 15k, rcl:R0805
- added R13: 1, rcl:R0805
- added R5: 22, rcl:R0805
- added R6, R7: 1.5k, rcl:R0805
- added R8: 330, rcl:R0805
- C4, C5: value (none) -> 22
- Q1: value (none) -> 12Mhz; device crystal-geyer_V1_0:3.2X2.5_KX-7 -> crystal:HC49/S
- moved C4 44.2 mm to (20.0, 29.5)
- moved C5 42.4 mm to (25.5, 29.5), turned to 180 degrees
- moved Q1 39.8 mm to (22.5, 25.5)
- moved R4 27.3 mm to (10.0, 16.5)
- moved R3 7.76 mm to (30.5, 21.4)
- moved U$1 4.95 mm to (43.0, 10.6), turned to 270 degrees
- moved U$2 3.89 mm to (22.6, 13.2)
- moved R1 3.20 mm to (15.0, 13.6)
- moved R2 3.04 mm to (10.0, 13.6)
- moved C6 2.00 mm to (11.0, 20.0)
- moved IC1 2.00 mm to (11.0, 26.0)
- moved C7 1.00 mm to (4.00, 26.0)
Connections:
- removed net VBUS: U$2.10
- removed net VCOM: U$2.18
- new net N$14: C1.2, R3.2, R4.2, U$2.21, U$2.25, U$2.26, U$2.4, U$2.7
- new net N$15: C10.2, R6.2
- new net N$16: C11.2, R7.2
- new net N$17: C11.1, C12.+, U$2.15
- new net N$18: C12.-, R9.1
- new net N$19: C13.-, R10.1
- new net N$20: C10.1, C13.+, U$2.14
- new net N$21: LED1.A, R8.1
- new net N$22: R10.2, R11.1, U$1.9
- new net N$23: R12.1, R9.2, U$1.11
- net +3V3: now also U$2.10
- net AGND: now also J1.1, R13.2; no longer U$1.4, U$2.12, U$2.17
- net GND: now also C1.1, C15.2, C2.2, C3.2, C8.2, C9.-, LED1.K, R13.1, R6.1, R7.1, U$1.4, U$2.11, U$2.12, U$2.17, U$2.19, U$2.6
- net N$10: now also C14.2
- net N$11: now also J1.5, R11.2, U$1.1; no longer U$1.9, U$2.14
- net N$12: now also J1.2, R12.2, U$1.14; no longer U$1.11, U$2.15
- net N$13: now also C15.1
- net N$3: now also C9.+, U$2.18; no longer R4.2, U$2.7
- net N$6: now also R4.1
- net N$7: now also Q1.2, R5.2; no longer Q1.1
- net N$8: now also Q1.1, R5.1; no longer Q1.3
- net N$9: now also C14.1
- net VCC: now also R8.2
- net VCCL: now also C3.1
- net VCCP: now also C2.1
- net VCCR: now also C8.1
Routing:
- net VCC: track 0.00 -> 88.2 mm
- net N$4: track 0.00 -> 34.8 mm
- net N$11: track 0.00 -> 33.0 mm
- net N$14: track 0.00 -> 30.6 mm
- net +3V3: track 0.00 -> 28.9 mm, vias 0 -> 2
- net N$19: track 0.00 -> 25.4 mm
- net N$18: track 0.00 -> 15.5 mm
- net N$7: track 0.00 -> 14.7 mm
- net N$8: track 0.00 -> 14.2 mm
- net N$13: track 0.00 -> 13.0 mm, vias 0 -> 2
- net N$23: track 0.00 -> 11.2 mm, vias 0 -> 2
- net N$22: track 0.00 -> 10.7 mm
- net N$5: track 0.00 -> 9.83 mm, vias 0 -> 2
- net N$12: track 0.00 -> 9.15 mm
- net N$2: track 0.00 -> 8.68 mm
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- added copper zone on layer 1, net AGND
- added copper zone on layer 16, net AGND
- added copper zone on layer 1, net GND
- added copper zone on layer 16, net GND

Commit message: Updated values
Parts:
- C2, C3, C8: value 22 -> 1u
- R11, R12: value 15k -> 22k
- R5: value 22 -> 1M
Changed lines of the file:
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@@
 <?xml version="1.0" encoding="utf-8"?>
 <!DOCTYPE eagle SYSTEM "eagle.dtd">
-<eagle version="8.4.1">
+<eagle version="8.7.0">
 <drawing>
 <settings>
@@
 <param name="checkRestrict" value="0"/>
 <param name="checkStop" value="0"/>
+<param name="checkValues" value="0"/>
 <param name="useDiameter" value="13"/>
 <param name="maxErrors" value="50"/>
@@
 <attribute name="SPICEPREFIX" value="C" x="4" y="26" size="1.778" layer="27" rot="R90" display="off"/>
 </element>
-<element name="R5" library="rcl" library_urn="urn:adsk.eagle:library:334" package="R0805" package3d_urn="urn:adsk.eagle:package:23553/2" value="22" x="22.5" y="21"/>
+<element name="R5" library="rcl" library_urn="urn:adsk.eagle:library:334" package="R0805" package3d_urn="urn:adsk.eagle:package:23553/2" value="1M" x="22.5" y="21"/>
 <element name="Q1" library="crystal" library_urn="urn:adsk.eagle:library:204" package="HC49/S" package3d_urn="urn:adsk.eagle:package:12071/1" value="12Mhz" x="22.5" y="25.5">
 <attribute name="MF" value="" x="22.5" y="25.5" size="1.778" layer="27" display="off"/>
@@
 <attribute name="SPICEPREFIX" value="C" x="30.5" y="18.5" size="1.778" layer="27" rot="R180" display="off"/>
 </element>
-<element name="C2" library="rcl" library_urn="urn:adsk.eagle:library:334" package="C0805" package3d_urn="urn:adsk.eagle:package:23617/2" value="22" x="30.5" y="15.5">
+<element name="C2" library="rcl" library_urn="urn:adsk.eagle:library:334" package="C0805" package3d_urn="urn:adsk.eagle:package:23617/2" value="1u" x="30.5" y="15.5">
 <attribute name="SPICEPREFIX" value="C" x="30.5" y="15.5" size="1.778" layer="27" display="off"/>
 </element>
-<element name="C3" library="rcl" library_urn="urn:adsk.eagle:library:334" package="C0805" package3d_urn="urn:adsk.eagle:package:23617/2" value="22" x="15" y="10.5" rot="R180">
+<element name="C3" library="rcl" library_urn="urn:adsk.eagle:library:334" package="C0805" package3d_urn="urn:adsk.eagle:package:23617/2" value="1u" x="15" y="10.5" rot="R180">
 <attribute name="SPICEPREFIX" value="C" x="15" y="10.5" size="1.778" layer="27" rot="R180" display="off"/>
 </element>
-<element name="C8" library="rcl" library_urn="urn:adsk.eagle:library:334" package="C0805" package3d_urn="urn:adsk.eagle:package:23617/2" value="22" x="30.5" y="8.5">
+<element name="C8" library="rcl" library_urn="urn:adsk.eagle:library:334" package="C0805" package3d_urn="urn:adsk.eagle:package:23617/2" value="1u" x="30.5" y="8.5">
 <attribute name="SPICEPREFIX" value="C" x="30.5" y="8.5" size="1.778" layer="27" display="off"/>
 </element>
@@
 <element name="R9" library="rcl" library_urn="urn:adsk.eagle:library:334" package="R0805" package3d_urn="urn:adsk.eagle:package:23553/2" value="10k" x="41" y="4.5" rot="R90"/>
 <element name="R10" library="rcl" library_urn="urn:adsk.eagle:library:334" package="R0805" package3d_urn="urn:adsk.eagle:package:23553/2" value="10k" x="44.5" y="4.5" rot="R90"/>
-<element name="R11" library="rcl" library_urn="urn:adsk.eagle:library:334" package="R0805" package3d_urn="urn:adsk.eagle:package:23553/2" value="15k" x="51.5" y="11" rot="R90"/>
-<element name="R12" library="rcl" library_urn="urn:adsk.eagle:library:334" package="R0805" package3d_urn="urn:adsk.eagle:package:23553/2" value="15k" x="48.5" y="11" rot="R90"/>
+<element name="R11" library="rcl" library_urn="urn:adsk.eagle:library:334" package="R0805" package3d_urn="urn:adsk.eagle:package:23553/2" value="22k" x="51.5" y="11" rot="R90"/>
+<element name="R12" library="rcl" library_urn="urn:adsk.eagle:library:334" package="R0805" package3d_urn="urn:adsk.eagle:package:23553/2" value="22k" x="48.5" y="11" rot="R90"/>
 <element name="R13" library="rcl" library_urn="urn:adsk.eagle:library:334" package="R0805" package3d_urn="urn:adsk.eagle:package:23553/2" value="1" x="35.5" y="29.5"/>
 </elements>
