File: usb-audio.sch (EAGLE design)
At the start: 12 parts

Commit message: .
Parts:
- removed C1, C2, C3: (no value), rcl:CPOL-EUA/3216-18R
- added C6: 10mF, rcl:CPOL-EUCT3216
- added C7: 100mF, rcl:CPOL-EUCT3216
- added IC1: LM1117MPX-3.3, lm1117:LM1117MPX-3.3
- added U$3: MICRO-USB, microusb:MICRO-USB
Connections:
- new net +3V3: C7.+, IC1.OUT, IC1.OUT1
- new net AGND: U$1.PGND, U$1.SGND, U$2.AGNDL, U$2.AGNDR
- new net GND: C4.2, C5.2, C6.-, C7.-, IC1.GND, U$3.GND, U$3.GND@1, U$3.GND@2
- new net N$10: U$1.C1N
- new net N$11: U$1.INL, U$2.VOUTL
- new net N$12: U$1.INR, U$2.VOUTR
- new net N$13: U$1.PVSS, U$1.SVSS
- new net N$5: R1.1, U$3.D-
- new net N$6: R2.1, U$3.D+
- new net N$7: C5.1, Q1.1, U$2.XTI
- new net N$8: C4.1, Q1.2, U$2.XTO
- new net N$9: U$1.C1P
- new net VCC: C6.+, IC1.IN, U$1.SHDN, U$1.VDD, U$3.VCC
Other:
- moved on the sheet: C4, C5, Q1, R1, R2, R3, R4, U$1, U$2

Commit message: rev 1
Parts:
- added C1: 100n, rcl:C-EUC0805
- added C10, C11, C2, C3, C8: 22, rcl:C-EUC0805
- added C12, C13: 220uF, rcl:CPOL-EUE2-5
- added C14, C15: 1uf, rcl:C-EUC0805
- added C9: 10mF, rcl:CPOL-EUCT3216
- added J1: PJ-324MH, audio:PJ-324MH
- added LED1: TLLR4400, led:TLLR4400
- added R10, R9: 10k, rcl:R-EU_R0805
- added R11, R12: 15k, rcl:R-EU_R0805
- added R13: 1, rcl:R-EU_R0805
- added R5: 22, rcl:R-EU_R0805
- added R6, R7: 1.5k, rcl:R-EU_R0805
- added R8: 330, rcl:R-EU_R0805
- C4, C5: value (none) -> 22
- Q1: value (none) -> 12Mhz; device crystal-geyer_V1_0:KX-7 -> crystal:CRYSTALHC49S
Connections:
- new net N$14: C1.2, R3.2, R4.2, U$2.HOST, U$2.PSEL, U$2.TEST0, U$2.TEST1, U$2.VDD
- new net N$15: C10.2, R6.2
- new net N$16: C11.2, R7.2
- new net N$17: C11.1, C12.+, U$2.VOUTR
- new net N$18: C12.-, R9.1
- new net N$19: C13.-, R10.1
- new net N$20: C10.1, C13.+, U$2.VOUTL
- new net N$21: LED1.A, R8.1
- new net N$22: R10.2, R11.1, U$1.INL
- new net N$23: R12.1, R9.2, U$1.INR
- new net VCCL: C3.1, U$2.VCCL
- new net VCCP: C2.1, U$2.VCCP
- new net VCCR: C8.1, U$2.VCCR
- net +3V3: now also U$2.VBUS
- net AGND: now also J1.1, R13.2; no longer U$1.PGND, U$2.AGNDL, U$2.AGNDR
- net GND: now also C1.1, C15.2, C2.2, C3.2, C8.2, C9.-, LED1.C, R13.1, R6.1, R7.1, U$1.PGND, U$2.AGNDL, U$2.AGNDR, U$2.DGND, U$2.PGND, U$2.ZGND
- net N$10: now also C14.2
- net N$11: now also J1.5, R11.2, U$1.OUTL; no longer U$1.INL, U$2.VOUTL
- net N$12: now also J1.2, R12.2, U$1.OUTR; no longer U$1.INR, U$2.VOUTR
- net N$13: now also C15.1
- net N$3: now also C9.+, U$2.VCOM; no longer R4.2, U$2.VDD
- net N$6: now also R4.1
- net N$7: now also Q1.2, R5.2; no longer Q1.1
- net N$8: now also Q1.1, R5.1; no longer Q1.2
- net N$9: now also C14.1
- net VCC: now also R8.2
Other:
- moved on the sheet: Q1, R1, R4

Commit message: Updated values
Parts:
- C2, C3, C8: value 22 -> 1u
- R11, R12: value 15k -> 22k
- R5: value 22 -> 1M
Changed lines of the file:
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@@
 <?xml version="1.0" encoding="utf-8"?>
 <!DOCTYPE eagle SYSTEM "eagle.dtd">
-<eagle version="8.4.1">
+<eagle version="8.7.0">
 <drawing>
 <settings>
@@
 <layer number="18" name="Vias" color="2" fill="1" visible="no" active="no"/>
 <layer number="19" name="Unrouted" color="6" fill="1" visible="no" active="no"/>
-<layer number="20" name="Dimension" color="15" fill="1" visible="no" active="no"/>
+<layer number="20" name="Dimension" color="24" fill="1" visible="no" active="no"/>
 <layer number="21" name="tPlace" color="7" fill="1" visible="no" active="no"/>
 <layer number="22" name="bPlace" color="7" fill="1" visible="no" active="no"/>
@@
 <part name="GND3" library="supply1" library_urn="urn:adsk.eagle:library:371" deviceset="GND" device=""/>
 <part name="P+4" library="supply1" library_urn="urn:adsk.eagle:library:371" deviceset="VCC" device=""/>
-<part name="R5" library="rcl" library_urn="urn:adsk.eagle:library:334" deviceset="R-EU_" device="R0805" package3d_urn="urn:adsk.eagle:package:23553/2" value="22"/>
+<part name="R5" library="rcl" library_urn="urn:adsk.eagle:library:334" deviceset="R-EU_" device="R0805" package3d_urn="urn:adsk.eagle:package:23553/2" value="1M"/>
 <part name="GND4" library="supply1" library_urn="urn:adsk.eagle:library:371" deviceset="GND" device=""/>
 <part name="GND5" library="supply1" library_urn="urn:adsk.eagle:library:371" deviceset="GND" device=""/>
@@
 <part name="GND7" library="supply1" library_urn="urn:adsk.eagle:library:371" deviceset="GND" device=""/>
 <part name="+3V1" library="supply1" library_urn="urn:adsk.eagle:library:371" deviceset="+3V3" device=""/>
-<part name="C2" library="rcl" library_urn="urn:adsk.eagle:library:334" deviceset="C-EU" device="C0805" package3d_urn="urn:adsk.eagle:package:23617/2" value="22"/>
-<part name="C3" library="rcl" library_urn="urn:adsk.eagle:library:334" deviceset="C-EU" device="C0805" package3d_urn="urn:adsk.eagle:package:23617/2" value="22"/>
-<part name="C8" library="rcl" library_urn="urn:adsk.eagle:library:334" deviceset="C-EU" device="C0805" package3d_urn="urn:adsk.eagle:package:23617/2" value="22"/>
+<part name="C2" library="rcl" library_urn="urn:adsk.eagle:library:334" deviceset="C-EU" device="C0805" package3d_urn="urn:adsk.eagle:package:23617/2" value="1u"/>
+<part name="C3" library="rcl" library_urn="urn:adsk.eagle:library:334" deviceset="C-EU" device="C0805" package3d_urn="urn:adsk.eagle:package:23617/2" value="1u"/>
+<part name="C8" library="rcl" library_urn="urn:adsk.eagle:library:334" deviceset="C-EU" device="C0805" package3d_urn="urn:adsk.eagle:package:23617/2" value="1u"/>
 <part name="GND8" library="supply1" library_urn="urn:adsk.eagle:library:371" deviceset="GND" device=""/>
 <part name="GND9" library="supply1" library_urn="urn:adsk.eagle:library:371" deviceset="GND" device=""/>
@@
 <part name="R9" library="rcl" library_urn="urn:adsk.eagle:library:334" deviceset="R-EU_" device="R0805" package3d_urn="urn:adsk.eagle:package:23553/2" value="10k"/>
 <part name="R10" library="rcl" library_urn="urn:adsk.eagle:library:334" deviceset="R-EU_" device="R0805" package3d_urn="urn:adsk.eagle:package:23553/2" value="10k"/>
-<part name="R11" library="rcl" library_urn="urn:adsk.eagle:library:334" deviceset="R-EU_" device="R0805" package3d_urn="urn:adsk.eagle:package:23553/2" value="15k"/>
-<part name="R12" library="rcl" library_urn="urn:adsk.eagle:library:334" deviceset="R-EU_" device="R0805" package3d_urn="urn:adsk.eagle:package:23553/2" value="15k"/>
+<part name="R11" library="rcl" library_urn="urn:adsk.eagle:library:334" deviceset="R-EU_" device="R0805" package3d_urn="urn:adsk.eagle:package:23553/2" value="22k"/>
+<part name="R12" library="rcl" library_urn="urn:adsk.eagle:library:334" deviceset="R-EU_" device="R0805" package3d_urn="urn:adsk.eagle:package:23553/2" value="22k"/>
 <part name="AGND2" library="supply1" library_urn="urn:adsk.eagle:library:371" deviceset="AGND" device=""/>
 <part name="GND18" library="supply1" library_urn="urn:adsk.eagle:library:371" deviceset="GND" device=""/>
@@
 packages will not be understood (or retained) with this version.
 </note>
-<note version="8.4" severity="warning">
-Since Version 8.4, EAGLE supports properties for SPICE simulation.
-Probes in schematics and SPICE mapping objects found in parts and library devices
-will not be understood with this version. Update EAGLE to the latest version
-for full support of SPICE simulation.
-</note>
 </compatibility>
